File: testpcb-edge-calibration/testpcb-edge-calibration.kicad_pcb (KiCad board)
At the start: 2 copper layers, 100 x 70 mm, 0 parts

Commit message: saving work
Routing:
- net (no net): track 23.2 -> 158.2 mm
